File: MCU.kicad_sch (KiCad schematic)
At the start: 14 parts, among them SW1 SW_Push, U1 ATmega328P-A, Y1 16MHz

Commit message: Pls check :)
Parts:
- C1, C2, C3, C4, C5, C6: footprint (none) -> Capacitor_SMD:C_0402_1005Metric
- L1: footprint (none) -> Inductor_SMD:L_0603_1608Metric
- R1, R2, R3, R4: footprint (none) -> Resistor_SMD:R_0402_1005Metric
- SW1: footprint (none) -> Button_Switch_SMD:SW_Push_SPST_NO_Alps_SKRK
- Y1: footprint (none) -> Crystal:Crystal_SMD_2012-2Pin_2.0x1.2mm
Connections:
- net SPI.SCLK renamed SPI.SCK
Changed lines of the file:
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@@
 		)
 	)
-	(global_label "GPIO_C{01,2,3,4,5}"
+	(global_label "GPIO_C{0,1,2,3,4,5}"
 		(shape input)
 		(at 248.92 17.78 180)
@@
 		)
 		(property "Intersheetrefs" "${INTERSHEET_REFS}"
-			(at 227.8523 17.78 0)
+			(at 227.2475 17.78 0)
 			(effects
 				(font
@@
 		)
 	)
-	(global_label "SPI{SS,MOSI,MISO,SCLK}"
+	(global_label "SPI{SS,MOSI,MISO,SCK}"
 		(shape input)
 		(at 252.73 34.29 180)
@@
 		)
 		(property "Intersheetrefs" "${INTERSHEET_REFS}"
-			(at 226.7637 34.29 0)
+			(at 227.7918 34.29 0)
 			(effects
 				(font
@@
 		)
 	)
-	(global_label "SPI.SCLK"
+	(global_label "SPI.SCK"
 		(shape input)
 		(at 109.22 80.01 0)
@@
 		)
 		(property "Intersheetrefs" "${INTERSHEET_REFS}"
-			(at 120.6719 80.01 0)
+			(at 119.6438 80.01 0)
 			(effects
 				(font
@@
 		)
 	)
-	(hierarchical_label "SPI{SS,MOSI,MISO,SCLK}"
+	(hierarchical_label "SPI{SS,MOSI,MISO,SCK}"
 		(shape input)
 		(at 257.81 34.29 0)
@@
 			)
 		)
-		(property "Footprint" ""
+		(property "Footprint" "Inductor_SMD:L_0603_1608Metric"
 			(at 102.87 59.69 0)
 			(effects
@@
 			)
 		)
-		(property "Footprint" ""
+		(property "Footprint" "Capacitor_SMD:C_0402_1005Metric"
 			(at 185.1152 69.85 0)
 			(effects
@@
 			)
 		)
-		(property "Footprint" ""
+		(property "Footprint" "Resistor_SMD:R_0402_1005Metric"
 			(at 129.032 100.33 90)
 			(effects
@@
 			)
 		)
-		(property "Footprint" ""
+		(property "Footprint" "Capacitor_SMD:C_0402_1005Metric"
 			(at 174.2948 62.23 0)
 			(effects
@@
 			)
 		)
-		(property "Footprint" ""
+		(property "Footprint" "Resistor_SMD:R_0402_1005Metric"
 			(at 182.372 101.6 90)
 			(effects
@@
 			)
 		)
-		(property "Footprint" ""
+		(property "Footprint" "Capacitor_SMD:C_0402_1005Metric"
 			(at 61.2648 67.31 0)
 			(effects
@@
 			)
 		)
-		(property "Footprint" ""
+		(property "Footprint" "Capacitor_SMD:C_0402_1005Metric"
 			(at 212.09 97.4852 0)
 			(effects
@@
 			)
 		)
-		(property "Footprint" ""
+		(property "Footprint" "Button_Switch_SMD:SW_Push_SPST_NO_Alps_SKRK"
 			(at 223.52 58.42 0)
 			(effects
@@
 			)
 		)
-		(property "Footprint" ""
+		(property "Footprint" "Resistor_SMD:R_0402_1005Metric"
 			(at 192.532 142.24 90)
 			(effects
@@
 			)
 		)
-		(property "Footprint" ""
+		(property "Footprint" "Capacitor_SMD:C_0402_1005Metric"
 			(at 212.09 106.3752 0)
 			(effects
@@
 			)
 		)
-		(property "Footprint" ""
+		(property "Footprint" "Resistor_SMD:R_0402_1005Metric"
 			(at 184.912 142.24 90)
 			(effects
@@
 			)
 		)
-		(property "Footprint" ""
+		(property "Footprint" "Crystal:Crystal_SMD_2012-2Pin_2.0x1.2mm"
 			(at 196.85 100.33 0)
 			(effects
@@
 			)
 		)
-		(property "Footprint" ""
+		(property "Footprint" "Capacitor_SMD:C_0402_1005Metric"
 			(at 124.46 58.7248 0)
 			(effects
