File: PSU.kicad_sch (KiCad schematic)
At the start: 19 parts, among them J1 USB_C_Receptacle_USB2.0_16P, U2 LM1117S-ADJ

Commit message: Pls check :)
Parts:
- C10, C9: footprint (none) -> Capacitor_SMD:CP_Elec_6.3x7.7
- C11: value 10u -> .1u; footprint (none) -> Capacitor_SMD:CP_Elec_6.3x7.7
- C7: footprint (none) -> Capacitor_SMD:C_0603_1608Metric
- C8: footprint (none) -> Capacitor_SMD:C_0402_1005Metric
- D3, D4: footprint (none) -> LED_SMD:LED_0402_1005Metric
- F1: footprint (none) -> Fuse:Fuse_1812_4532Metric
- FB1: footprint (none) -> Inductor_SMD:L_0603_1608Metric
- J1: footprint (none) -> Connector_USB:USB_C_Receptacle_Palconn_UTC16-G
- R10, R5, R6, R7, R8, R9: footprint (none) -> Resistor_SMD:R_0402_1005Metric
- U2: footprint Package_TO_SOT_SMD:TO-263-3_TabPin2 -> Package_TO_SOT_SMD:SOT-223
Changed lines of the file:
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@@
 	)
 	(junction
+		(at 81.28 147.32)
+		(diameter 0)
+		(color 0 0 0 0)
+	)
+	(junction
 		(at 59.69 147.32)
 		(diameter 0)
@@
 		(color 0 0 0 0)
 	)
-	(junction
-		(at 85.09 147.32)
-		(diameter 0)
-		(color 0 0 0 0)
-	)
 	(no_connect
 		(at 77.47 87.63)
@@
 	(wire
 		(pts
+			(xy 81.28 157.48) (xy 81.28 161.29)
+		)
+		(stroke
+			(width 0)
+			(type default)
+		)
+	)
+	(wire
+		(pts
 			(xy 99.06 154.94) (xy 99.06 158.75)
 		)
@@
 	(wire
 		(pts
-			(xy 76.2 147.32) (xy 85.09 147.32)
+			(xy 76.2 147.32) (xy 81.28 147.32)
 		)
 		(stroke
@@
 	(wire
 		(pts
-			(xy 195.58 54.61) (xy 195.58 55.88)
+			(xy 81.28 147.32) (xy 99.06 147.32)
 		)
 		(stroke
@@
 	(wire
 		(pts
-			(xy 80.01 72.39) (xy 80.01 99.06)
+			(xy 195.58 54.61) (xy 195.58 55.88)
 		)
 		(stroke
@@
 	(wire
 		(pts
-			(xy 170.18 71.12) (xy 170.18 81.28)
+			(xy 80.01 72.39) (xy 80.01 99.06)
 		)
 		(stroke
@@
 	(wire
 		(pts
-			(xy 204.47 71.12) (xy 204.47 80.01)
+			(xy 170.18 71.12) (xy 170.18 81.28)
 		)
 		(stroke
@@
 	(wire
 		(pts
-			(xy 171.45 127) (xy 171.45 132.08)
+			(xy 204.47 71.12) (xy 204.47 80.01)
 		)
 		(stroke
@@
 	(wire
 		(pts
-			(xy 85.09 147.32) (xy 99.06 147.32)
+			(xy 171.45 127) (xy 171.45 132.08)
 		)
 		(stroke
@@
 	(wire
 		(pts
-			(xy 85.09 154.94) (xy 85.09 158.75)
+			(xy 81.28 147.32) (xy 81.28 149.86)
 		)
 		(stroke
@@
 			)
 		)
-		(property "Footprint" ""
+		(property "Footprint" "Fuse:Fuse_1812_4532Metric"
 			(at 124.46 146.05 0)
 			(effects
@@
 			)
 		)
-		(property "Footprint" ""
+		(property "Footprint" "Resistor_SMD:R_0402_1005Metric"
 			(at 169.672 123.19 90)
 			(effects
@@
 			)
 		)
-		(property "Value" "10u"
+		(property "Value" ".1u"
 			(at 207.01 69.4181 0)
 			(effects
@@
 			)
 		)
-		(property "Footprint" ""
+		(property "Footprint" "Capacitor_SMD:CP_Elec_6.3x7.7"
 			(at 204.47 68.58 0)
 			(effects
@@
 			)
 		)
-		(property "Footprint" "Package_TO_SOT_SMD:TO-263-3_TabPin2"
+		(property "Footprint" "Package_TO_SOT_SMD:SOT-223"
 			(at 184.15 54.61 0)
 			(effects
@@
 			)
 		)
-		(property "Footprint" ""
+		(property "Footprint" "Resistor_SMD:R_0402_1005Metric"
 			(at 111.252 67.31 90)
 			(effects
@@
 	(symbol
 		(lib_id "power:GND")
+		(at 81.28 161.29 0)
+		(unit 1)
+		(exclude_from_sim no)
+		(in_bom yes)
+		(on_board yes)
+		(dnp no)
+		(fields_autoplaced yes)
+		(property "Reference" "#PWR024"
+			(at 81.28 167.64 0)
+			(effects
+				(font
+					(size 1.27 1.27)
+				)
+				(hide yes)
+			)
+		)
+		(property "Value" "GND"
+			(at 81.28 166.37 0)
+			(effects
+				(font
+					(size 1.27 1.27)
+				)
+			)
+		)
+		(property "Footprint" ""
+			(at 81.28 161.29 0)
+			(effects
+				(font
+					(size 1.27 1.27)
+				)
+				(hide yes)
+			)
+		)
+		(property "Datasheet" ""
+			(at 81.28 161.29 0)
+			(effects
+				(font
+					(size 1.27 1.27)
+				)
+				(hide yes)
+			)
+		)
+		(property "Description" "Power symbol creates a global label with name \"GND\" , ground"
+			(at 81.28 161.29 0)
+			(effects
+				(font
+					(size 1.27 1.27)
+				)
+				(hide yes)
+			)
+		)
+		(pin "1"
+		)
+		(instances
+			(project "Socet_Onboarding"
+				(path "/4f6ede97-95f2-479b-8a62-4dd4f1f7b83b/c73a435e-84d1-47f3-96bd-7afc98a52d98"
+					(reference "#PWR024")
+					(unit 1)
+				)
+			)
+		)
+	)
+	(symbol
+		(lib_id "power:GND")
 		(at 80.01 109.22 0)
 		(unit 1)
@@
 			)
 		)
-		(property "Footprint" ""
+		(property "Footprint" "Connector_USB:USB_C_Receptacle_Palconn_UTC16-G"
 			(at 66.04 72.39 0)
 			(effects
@@
 			)
 		)
-		(property "Footprint" ""
+		(property "Footprint" "Resistor_SMD:R_0402_1005Metric"
 			(at 193.802 72.39 90)
 			(effects
@@
 			)
 		)
-		(property "Footprint" ""
+		(property "Footprint" "Capacitor_SMD:C_0603_1608Metric"
 			(at 58.7248 147.32 0)
 			(effects
@@
 			)
 		)
-		(property "Footprint" ""
+		(property "Footprint" "Resistor_SMD:R_0402_1005Metric"
 			(at 193.802 59.69 90)
 			(effects
@@
 			)
 		)
-		(property "Footprint" ""
+		(property "Footprint" "Capacitor_SMD:CP_Elec_6.3x7.7"
 			(at 170.18 68.58 0)
 			(effects
@@
 			)
 		)
-		(property "Footprint" ""
+		(property "Footprint" "Resistor_SMD:R_0402_1005Metric"
 			(at 183.642 121.92 90)
 			(effects
@@
 			)
 		)
-		(property "Footprint" ""
+		(property "Footprint" "LED_SMD:LED_0402_1005Metric"
 			(at 171.45 135.89 0)
 			(effects
@@
 	(symbol
 		(lib_id "Device:C")
-		(at 85.09 151.13 180)
+		(at 81.28 153.67 180)
 		(unit 1)
 		(exclude_from_sim no)
@@
 		(fields_autoplaced yes)
 		(property "Reference" "C8"
-			(at 88.9 149.8599 0)
+			(at 85.09 152.3999 0)
 			(effects
 				(font
@@
 		)
 		(property "Value" "0.1u"
-			(at 88.9 152.3999 0)
+			(at 85.09 154.9399 0)
 			(effects
 				(font
@@
 			)
 		)
-		(property "Footprint" ""
-			(at 84.1248 147.32 0)
+		(property "Footprint" "Capacitor_SMD:C_0402_1005Metric"
+			(at 80.3148 149.86 0)
 			(effects
 				(font
@@
 		)
 		(property "Datasheet" "~"
-			(at 85.09 151.13 0)
+			(at 81.28 153.67 0)
 			(effects
 				(font
@@
 		)
 		(property "Description" "Unpolarized capacitor"
-			(at 85.09 151.13 0)
+			(at 81.28 153.67 0)
 			(effects
 				(font
@@
 			)
 		)
-		(property "Footprint" ""
+		(property "Footprint" "Resistor_SMD:R_0402_1005Metric"
 			(at 99.822 68.58 90)
 			(effects
@@
 			)
 		)
-		(property "Footprint" ""
+		(property "Footprint" "Capacitor_SMD:CP_Elec_6.3x7.7"
 			(at 100.0252 154.94 0)
 			(effects
@@
 	(symbol
 		(lib_id "power:GND")
-		(at 85.09 158.75 0)
-		(unit 1)
-		(exclude_from_sim no)
-		(in_bom yes)
-		(on_board yes)
-		(dnp no)
-		(fields_autoplaced yes)
-		(property "Reference" "#PWR024"
-			(at 85.09 165.1 0)
-			(effects
-				(font
-					(size 1.27 1.27)
-				)
-				(hide yes)
-			)
-		)
-		(property "Value" "GND"
-			(at 85.09 163.83 0)
-			(effects
-				(font
-					(size 1.27 1.27)
-				)
-			)
-		)
-		(property "Footprint" ""
-			(at 85.09 158.75 0)
-			(effects
-				(font
-					(size 1.27 1.27)
-				)
-				(hide yes)
-			)
-		)
-		(property "Datasheet" ""
-			(at 85.09 158.75 0)
-			(effects
-				(font
-					(size 1.27 1.27)
-				)
-				(hide yes)
-			)
-		)
-		(property "Description" "Power symbol creates a global label with name \"GND\" , ground"
-			(at 85.09 158.75 0)
-			(effects
-				(font
-					(size 1.27 1.27)
-				)
-				(hide yes)
-			)
-		)
-		(pin "1"
-		)
-		(instances
-			(project "Socet_Onboarding"
-				(path "/4f6ede97-95f2-479b-8a62-4dd4f1f7b83b/c73a435e-84d1-47f3-96bd-7afc98a52d98"
-					(reference "#PWR024")
-					(unit 1)
-				)
-			)
-		)
-	)
-	(symbol
-		(lib_id "power:GND")
 		(at 113.03 74.93 0)
 		(unit 1)
@@
 			)
 		)
-		(property "Footprint" ""
+		(property "Footprint" "Inductor_SMD:L_0603_1608Metric"
 			(at 72.39 149.098 90)
 			(effects
@@
 			)
 		)
-		(property "Footprint" ""
+		(property "Footprint" "LED_SMD:LED_0402_1005Metric"
 			(at 185.42 134.62 0)
 			(effects
