File: Peripherals .kicad_sch (KiCad schematic)
At the start: 3 parts, among them J2 Conn_01x16_Socket, J3 Conn_01x16_Socket, J4 ICSP

Commit message: Pls check :)
Parts:
- J2, J3: footprint (none) -> Connector_PinHeader_2.54mm:PinHeader_1x16_P2.54mm_Vertical
- J4: footprint (none) -> Connector_PinSocket_2.54mm:PinSocket_2x03_P2.54mm_Vertical
Changed lines of the file:
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@@
 		)
 	)
-	(global_label "SPI{SS,MOSI,MISO,SCLK}"
+	(global_label "SPI{SS,MOSI,MISO,SCK}"
 		(shape input)
 		(at 251.46 35.56 180)
@@
 		)
 		(property "Intersheetrefs" "${INTERSHEET_REFS}"
-			(at 225.4937 35.56 0)
+			(at 226.5218 35.56 0)
 			(effects
 				(font
@@
 		)
 	)
-	(global_label "GPIO_C{01,2,3,4,5}"
+	(global_label "GPIO_C{0,1,2,3,4,5}"
 		(shape input)
 		(at 246.38 17.78 180)
@@
 		)
 		(property "Intersheetrefs" "${INTERSHEET_REFS}"
-			(at 225.3123 17.78 0)
+			(at 224.7075 17.78 0)
 			(effects
 				(font
@@
 		)
 	)
-	(hierarchical_label "SPI{SS,MOSI,MISO,SLCK}"
+	(hierarchical_label "SPI{SS,MOSI,MISO,SCK}"
 		(shape input)
 		(at 257.81 35.56 0)
@@
 			)
 		)
-		(property "Footprint" ""
+		(property "Footprint" "Connector_PinHeader_2.54mm:PinHeader_1x16_P2.54mm_Vertical"
 			(at 127 99.06 0)
 			(effects
@@
 			)
 		)
-		(property "Footprint" ""
+		(property "Footprint" "Connector_PinHeader_2.54mm:PinHeader_1x16_P2.54mm_Vertical"
 			(at 106.68 96.52 0)
 			(effects
@@
 			)
 		)
-		(property "Footprint" ""
+		(property "Footprint" "Connector_PinSocket_2.54mm:PinSocket_2x03_P2.54mm_Vertical"
 			(at 204.47 72.39 0)
 			(effects
