File: Socet_Onboarding.kicad_sch (KiCad schematic)
At the start: 0 parts

Commit message: Pls check :)
Other:
- sheet MCU ports: added SPI{SS,MOSI,MISO,SCK}; removed SPI{SS,MOSI,MISO,SCLK}
- sheet Peripherals ports: added SPI{SS,MOSI,MISO,SCK}; removed SPI{SS,MOSI,MISO,SLCK}
Changed lines of the file:
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@@
 			)
 		)
-		(pin "SPI{SS,MOSI,MISO,SLCK}" input
+		(pin "SPI{SS,MOSI,MISO,SCK}" input
 			(at 245.618 64.77 0)
 			(effects
@@
 			)
 		)
-		(pin "SPI{SS,MOSI,MISO,SCLK}" input
+		(pin "SPI{SS,MOSI,MISO,SCK}" input
 			(at 252.222 121.92 0)
 			(effects
