File: Socet_Onboarding.kicad_pcb (KiCad board)
At the start: 2 copper layers, 83.7 x 44.5 mm, 45 parts, among them J1 USB_C_Receptacle_USB2.0_16P, J2 Conn_01x16_Socket, J3 Conn_01x16_Socket, J4 ICSP, SW1 SW_Push, U1 ATmega328P-A, U2 LM1117S-ADJ, U3 FT232RL, Y1 16MHz

Commit message: 0 Errors except the ones to ignore I think 0 warnings
Other:
- board size 83.7 x 44.5 mm -> 97.1 x 53.8 mm
Changed lines of the file:
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@@
 	)
 	(gr_rect
-		(start 101.7 69.95)
-		(end 185.4 114.45)
+		(start 96.7 64.9)
+		(end 193.8 118.7)
 		(stroke
 			(width 0.05)
